Commit message: feat: 更新Cello模型文件和URDF参数，调整了URDF中link7的位置

File: src/cello_description/urdf/cello_description.urdf (robot description, URDF)
Before this commit: robot cello_description, 10 links, 9 joints
Links:
- link base_link: mass 0.860146104012974 -> 0.860146103977898
- link link6: mass 0.0539231941559604 -> 0.053923
- link link7_left: mass 0.0118967398398553 -> 0.011897
- link link7_right: mass 0.0118967398398553 -> 0.011897
Joints:
- joint joint3: origin xyz=0.2476 -0.0396 0 rpy=0 0 -1.5708 -> xyz=0.24760456425896 -0.0395999999999958 0 rpy=0 0 -1.5707963267949
- joint joint6: origin xyz=-0.00132500000000002 -0.170658355416465 0 rpy=1.5707963267949 -1.5707963267949 0 -> xyz=-0.001325 -0.17066 0 rpy=1.5708 -1.5708 0
- joint joint7_left: origin xyz=0 0.0136874999999999 0 rpy=1.5707963267949 0 -1.5707963267949 -> xyz=0 0.013687 0.01825 rpy=1.5708 0 -1.5708
- joint joint7_right: origin xyz=0 0.0136874999999999 0 rpy=1.5707963267949 0 -1.5707963267949 -> xyz=0 0.013687 0.01825 rpy=1.5708 0 -1.5708

File: src/cello_gazebo/urdf/cello_gazebo.urdf (robot description, URDF)
Before this commit: robot cello_description, 9 links, 8 joints
Links:
- link base_link: mass 0.860146104031393 -> 0.860146103977898
- link link1: mass 0.211492634096808 -> 0.21149263410611
- link link2: mass 0.226428575789942 -> 0.226428575799244
- link link6: mass 0.0539231941559604 -> 0.053923
- link link7_left: mass 0.0118967398398553 -> 0.011897
- link link7_right: mass 0.0118967398398553 -> 0.011897
Joints:
- joint joint1: origin xyz=0 0 0.0665 rpy=0 0 3.14159265358979 -> xyz=0 0 0.0635 rpy=0 0 0
- joint joint2: origin xyz=0.0022 0 0.0638 rpy=1.5708 -1.5708 0 -> xyz=0.00220000000000002 0 0.0638 rpy=1.5707963267949 -1.5707963267949 0
- joint joint3: origin xyz=0.2476 -0.0396 0 rpy=0 0 -1.5708 -> xyz=0.24760456425896 -0.0395999999999958 0 rpy=0 0 -1.5707963267949
- joint joint4: origin xyz=0.26712 -0.00308 0 rpy=1.5708 0 1.5708 -> xyz=0.267124999999999 -0.00308000000000425 0 rpy=1.5707963267949 0 1.5707963267949
- joint joint5: origin xyz=0 0 0 rpy=-1.5708 0 0 -> xyz=0 0 0 rpy=-1.5707963267949 0 0
- joint joint7_left: origin xyz=0 0.013687 0 rpy=1.5708 0 -1.5708 -> xyz=0 0.013687 0.01825 rpy=1.5708 0 -1.5708
- joint joint7_right: origin xyz=0 0.013687 0 rpy=1.5708 0 -1.5708 -> xyz=0 0.013687 0.01825 rpy=1.5708 0 -1.5708
