Commit message: Merge branch 'GTC_demo_fixes'

File: src/cello_moveit_config/config/camera_with_stand.xacro (robot description, xacro)
@@ -1,5 +1,7 @@
 <?xml version="1.0"?>
 <robot xmlns:xacro="http://ros.org/wiki/xacro" >
-    <xacro:macro name="camera_with_stand" params="camera_pos_z camera_type:=realsense">
+    <xacro:macro name="camera_with_stand" params="camera_pos_z
+                                                  camera_roll:=0.0 camera_pitch:=0.0 camera_yaw:=0.0
+                                                  camera_type:=realsense">
         <!-- Variables -->
         <xacro:property name="pi_val" value="3.1415926535"/>
@@ -13,4 +15,5 @@
         </xacro:if>
         <!-- Links -->
+        <link name="camera_mount_link"/>
         <link name="camera_base_link"/>
         <xacro:if value="${camera_type != 'realsense'}">
@@ -65,4 +68,9 @@
         </link>
         <!-- Joints -->
+        <joint name="camera_mount_camera_base_joint" type="fixed">
+            <parent link="camera_mount_link"/>
+            <child link="camera_base_link"/>
+            <origin xyz="0 0 0" rpy="${camera_roll} ${camera_pitch} ${camera_yaw}"/>
+        </joint>
         <xacro:if value="${camera_type == 'realsense'}">
             <xacro:sensor_d435i parent="camera_base_link" use_nominal_extrinsics="true" >
@@ -78,7 +86,7 @@
         </xacro:if>
         <joint name="camera_base_to_upper_arm_joint" type="fixed">
-            <parent link="camera_base_link"/>
+            <parent link="camera_mount_link"/>
             <child link="camera_holder_upper_arm_link"/>
-            <origin xyz="-0.03 0 0.0125" rpy="0 0 0"/>
+            <origin xyz="-0.0125 0 0.03" rpy="${pi_val} ${pi_val/2} 0"/>
         </joint>
         <joint name="camera_holder_upper_arm_to_camera_holder_lower_arm_joint" type="fixed">

File: src/cello_moveit_config/config/cello_description.urdf.xacro (robot description, xacro)
@@ -3,9 +3,9 @@
     <!-- Arguments -->
     <xacro:arg name="initial_positions_file" default="initial_positions.yaml" />
-    <xacro:arg name="launch_camera" default="false" />
+    <xacro:arg name="launch_camera" default="true" />
     <xacro:arg name="camera_type" default="realsense" />
-    <xacro:arg name="camera_pos_x" default="0.25" />
+    <xacro:arg name="camera_pos_x" default="0.4" />
     <xacro:arg name="camera_pos_y" default="0.0" />
-    <xacro:arg name="camera_pos_z" default="0.4" />
+    <xacro:arg name="camera_pos_z" default="0.68" />
     <xacro:arg name="camera_pos_roll" default="0.0" />
     <xacro:arg name="camera_pos_pitch" default="1.57079633" />
@@ -19,11 +19,13 @@
     <xacro:if value="$(eval launch_camera)">
         <xacro:include filename="$(find cello_moveit_config)/config/camera_with_stand.xacro"/>
-        <xacro:camera_with_stand camera_pos_z="$(arg camera_pos_z)" camera_type="$(arg camera_type)" />
+        <xacro:camera_with_stand camera_pos_z="$(arg camera_pos_z)"
+                                 camera_roll="$(arg camera_pos_roll)" camera_pitch="$(arg camera_pos_pitch)" camera_yaw="$(arg camera_pos_yaw)"
+                                 camera_type="$(arg camera_type)" />
         <!-- Connect camera to robot base -->
-        <joint name="base_link_camera_base_joint" type="fixed">
+        <joint name="base_link_camera_mount_joint" type="fixed">
             <parent link="base_link"/>
-            <child link="camera_base_link"/>
+            <child link="camera_mount_link"/>
             <origin xyz="$(arg camera_pos_x) $(arg camera_pos_y) $(arg camera_pos_z)"
-                    rpy="$(arg camera_pos_roll) $(arg camera_pos_pitch) $(arg camera_pos_yaw)"/>
+                    rpy="0 0 0"/>
         </joint>
     </xacro:if>
