Commit message: calibrated tf path correction

File: src/viola_moveit_config/config/calibrated_camera_with_stand.urdf.xacro (robot description, xacro)
@@ -1,5 +1,5 @@
 <?xml version="1.0"?>
 <robot xmlns:xacro="http://www.ros.org/wiki/xacro" name="calibrated_camera_with_stand">
-    <xacro:arg name="camera_name" default="realsense" />
+    <xacro:arg name="camera_name" default="camera" />
     <xacro:arg name="camera_pos_z" default="0.64" />
     <xacro:arg name="camera_pos_roll" default="-0.03" />
@@ -7,5 +7,5 @@
     <xacro:arg name="camera_pos_yaw" default="3.14159265" />
     <xacro:include filename="$(find viola_moveit_config)/config/camera_with_stand.xacro"/>
-    <link name="camera_color_optical_frame"/>
+    <link name="realsense_color_optical_frame"/>
     <xacro:camera_with_stand camera_pos_z="$(arg camera_pos_z)"
                              camera_roll="$(arg camera_pos_roll)"
@@ -14,8 +14,8 @@
                              camera_name="$(arg camera_name)" />
     <joint name="camera_color_optical_frame_to_camera_connection_joint" type="fixed">
-        <parent link="camera_color_optical_frame"/>
+        <parent link="realsense_color_optical_frame"/>
         <child link="camera_connection_link"/>
-        <origin xyz="0.033 0.012 -0.011"
-                rpy="0.785 -1.571 0.000"/>
+        <origin xyz="0.0325 0.0125 -0.0106"
+                rpy="1.5707963268 -1.5707963268 0"/>
     </joint>
 </robot>

File: src/viola_moveit_config/config/viola_description.urdf.xacro (robot description, xacro)
@@ -6,5 +6,5 @@
     <xacro:arg name="use_camera_calibration" default="false" />
     <xacro:arg name="launch_camera" default="false" />
-    <xacro:arg name="camera_name" default="realsense" />
+    <xacro:arg name="camera_name" default="camera" />
     <xacro:arg name="camera_pos_x" default="0.4" />
     <xacro:arg name="camera_pos_y" default="0.0" />

Commit message: calibration_board_holder only during calibration

File: src/viola_moveit_config/config/calibrated_camera_with_stand.urdf.xacro (robot description, xacro)
@@ -13,5 +13,5 @@
                              camera_yaw="$(arg camera_pos_yaw)"
                              camera_name="$(arg camera_name)" />
-    <joint name="camera_color_optical_frame_to_camera_connection_joint" type="fixed">
+    <joint name="realsense_color_optical_frame_to_camera_connection_joint" type="fixed">
         <parent link="realsense_color_optical_frame"/>
         <child link="camera_connection_link"/>

File: src/viola_moveit_config/config/camera_with_stand.xacro (robot description, xacro)
@@ -11,5 +11,5 @@
                                                   camera_pitch:=0.0
                                                   camera_yaw:=0.0
-                                                  camera_name:=realsense">
+                                                  camera_name:=camera">
         <!-- Include realsense urdf macro -->
         <xacro:include filename="$(find realsense2_description)/urdf/_d435i.urdf.xacro"/>

File: src/viola_moveit_config/config/viola_description.urdf.xacro (robot description, xacro)
@@ -3,5 +3,5 @@
     <!-- Arguments -->
     <xacro:arg name="initial_positions_file" default="initial_positions.yaml" />
-    <xacro:arg name="launch_calibration" default="true" />
+    <xacro:arg name="launch_calibration" default="false" />
     <xacro:arg name="use_camera_calibration" default="false" />
     <xacro:arg name="launch_camera" default="false" />
