Commit message: add calibration plate to urdf & modify launch arguments
Co-authored-by: Copilot <copilot@github.com>

File: src/viola_description/urdf/viola_description.urdf (robot description, URDF)
Before this commit: robot viola_description, 10 links, 9 joints
Links:
- added link calib_connection_link
Joints:
- added joint link6_to_calib_connection_joint: type fixed, parent link6, child calib_connection_link, origin xyz=0 -0.022 -0.054 rpy=0 0 0

File: src/viola_moveit_config/config/viola_description.urdf.xacro (robot description, xacro)
@@ -3,5 +3,6 @@
     <!-- Arguments -->
     <xacro:arg name="initial_positions_file" default="initial_positions.yaml" />
-    <xacro:arg name="launch_camera" default="true" />
+    <xacro:arg name="launch_calibration" default="true" />
+    <xacro:arg name="launch_camera" default="false" />
     <xacro:arg name="camera_type" default="realsense" />
     <xacro:arg name="camera_pos_x" default="0.4" />
@@ -16,7 +17,7 @@
     <xacro:include filename="viola_description.ros2_control.xacro" />
     <xacro:viola_description_ros2_control name="FakeSystem" initial_positions_file="$(arg initial_positions_file)"/>
-    <!-- Conditionally include control if not GUI -->
+    <!-- Conditionally include camera-->
     <xacro:if value="$(eval launch_camera)">
-        <xacro:include filename="$(find cello_moveit_config)/config/camera_with_stand.xacro"/>
+        <xacro:include filename="$(find viola_moveit_config)/config/camera_with_stand.xacro"/>
         <xacro:camera_with_stand camera_pos_z="$(arg camera_pos_z)"
                                  camera_roll="$(arg camera_pos_roll)" camera_pitch="$(arg camera_pos_pitch)" camera_yaw="$(arg camera_pos_yaw)"
@@ -30,3 +31,8 @@
         </joint>
     </xacro:if>
+    <!-- Conditionally include calibration plate-->
+    <xacro:if value="$(eval launch_calibration)">
+        <xacro:include filename="$(find viola_moveit_config)/config/calibration_board_holder.xacro"/>
+        <xacro:calibration_board_holder parent="calib_connection_link"/>
+    </xacro:if>
 </robot>
